File: Sorcerer/MasterVideoTiming.kicad_sch (KiCad schematic)
At the start: 27 parts, among them J14 Jumper, J15 Jumper, J18 Jumper, U1 74LS74, Y1 12.638MHz

Commit message: Fix some issues I found.
Connections:
- net 5CLK6: no longer C1.1, R2.2, U1.10 (~{S}), U1.13 (~{R}), UA3.1 (~{MR}), UA3.10 (CET), UA3.7 (CEP), UA4.1 (~{MR}), UA5.15 (~{R}), UA5.4 (~{S}), UB1.1 (~{R}), UB1.10 (~{S}), UB1.4 (~{S}), UB3.1 (~{MR}), UB3.10 (CET), UB3.7 (CEP), UB4.1 (~{MR}), UB5.10 (~{S}), UB5.12 (K), UB5.14 (~{R}), UB5.15 (~{R}), UB5.2 (K), UB5.4 (~{S}), UB6.11 (I0b), UB7.1 (~{R}), UB7.13 (~{R})
- new net V_PUP: C1.1, R2.2, U1.10 (~{S}), U1.13 (~{R}), UA3.1 (~{MR}), UA3.10 (CET), UA3.7 (CEP), UA4.1 (~{MR}), UA5.15 (~{R}), UA5.4 (~{S}), UB1.1 (~{R}), UB1.10 (~{S}), UB1.4 (~{S}), UB3.1 (~{MR}), UB3.10 (CET), UB3.7 (CEP), UB4.1 (~{MR}), UB5.10 (~{S}), UB5.12 (K), UB5.14 (~{R}), UB5.15 (~{R}), UB5.2 (K), UB5.4 (~{S}), UB6.11 (I0b), UB7.1 (~{R}), UB7.13 (~{R})
Changed lines of the file:
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@@
-	)
-	(junction
-		(at 347.98 175.26)
-		(diameter 0)
-		(color 0 0 0 0)
 	)
 	(junction
@@
 	(wire
 		(pts
-			(xy 339.09 180.34) (xy 339.09 175.26)
+			(xy 339.09 180.34) (xy 339.09 173.99)
 		)
 		(stroke
@@
 	(wire
 		(pts
+			(xy 339.09 173.99) (xy 358.14 173.99)
+		)
+		(stroke
+			(width 0)
+			(type default)
+		)
+	)
+	(wire
+		(pts
 			(xy 121.92 196.85) (xy 125.73 196.85)
 		)
@@
 	(wire
 		(pts
-			(xy 339.09 175.26) (xy 347.98 175.26)
-		)
-		(stroke
-			(width 0)
-			(type default)
-		)
-	)
-	(wire
-		(pts
 			(xy 67.31 55.88) (xy 67.31 135.89)
 		)
@@
 	(wire
 		(pts
-			(xy 358.14 175.26) (xy 358.14 185.42)
+			(xy 358.14 173.99) (xy 358.14 185.42)
 		)
 		(stroke
@@
 		)
 		(stroke
-			(width 0)
-			(type default)
-		)
-	)
-	(wire
-		(pts
-			(xy 347.98 175.26) (xy 358.14 175.26)
-		)
-		(stroke
