File: Sorcerer/VideoInterface.kicad_sch (KiCad schematic)
At the start: 31 parts, among them J4 VIDEO, Q1 2N2222

Commit message: Fix some issues I found.
Parts:
- J4: value VIDEO -> AV-103B
Changed lines of the file:
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@@
 			)
 		)
-		(property "Value" "VIDEO"
+		(property "Value" "AV-103B"
 			(at 401.32 65.0631 0)
 			(effects
