File: Sorcerer/dynamic_ram.kicad_sch (KiCad schematic)
At the start: 36 parts, among them J5 Jumper, J6 Jumper

Commit message: Fix some issues I found.
Connections:
- net 4K/16K renamed 4K/~{16K}
Changed lines of the file:
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@@
 		)
 	)
-	(label "4K{slash}16K"
+	(label "4K{slash}~{16K}"
 		(at 101.6 209.55 0)
 		(effects

Commit message: Minor fixes.
Connections:
- net ~{DRAS1}: now also UB11.1, UC10.7 (Za)
- net ~{DRAS2}: now also UB11.2, UC10.9 (Zb)
Changed lines of the file:
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@@
+		)
+	)
+	(global_label "~{DRAS1}"
+		(shape input)
+		(at 166.37 195.58 90)
+		(fields_autoplaced yes)
+		(effects
+			(font
+				(size 1.27 1.27)
+			)
+			(justify left)
+		)
+		(property "Intersheetrefs" "${INTERSHEET_REFS}"
+			(at 166.37 186.5472 90)
+			(effects
+				(font
+					(size 1.27 1.27)
+				)
+				(justify left)
+				(hide yes)
+			)
 		)
 	)
@@
 			(effects
 				(font
+					(size 1.27 1.27)
+				)
+				(justify right)
+				(hide yes)
+			)
+		)
+	)
+	(global_label "~{DRAS2}"
+		(shape input)
+		(at 166.37 207.01 180)
+		(fields_autoplaced yes)
+		(effects
+			(font
+				(size 1.27 1.27)
+			)
+			(justify right)
+		)
+		(property "Intersheetrefs" "${INTERSHEET_REFS}"
+			(at 157.3372 207.01 0)
+			(effects
+				(font
