File: Sorcerer/interfaces.kicad_sch (KiCad schematic)
At the start: 54 parts, among them J13 Amp Connector, J16 Mic 1 Jack, J17 Ear Jack, J2 Parallel Port, J3 S100, Q2 2N2222, Q3 2N2222

Commit message: Minor fixes.
Parts:
- J2: value Parallel Port -> Serial Port
Changed lines of the file:
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@@
 			)
 		)
-		(property "Value" "Parallel Port"
+		(property "Value" "Serial Port"
 			(at 152.4 95.2499 0)
 			(effects
